Commit message: Robot with basic URDF

File: mobile_robot/urdf/rover.urdf (robot description, URDF)
Before this commit: robot rover, 1 links, 0 joints
Links:
- added link base_footprint
- added link front_left_wheel; collision cylinder length=0.1 radius=0.15; visual cylinder length=0.1 radius=0.15
- added link front_right_wheel; collision cylinder length=0.1 radius=0.15; visual cylinder length=0.1 radius=0.15
- added link rear_left_wheel; collision cylinder length=0.1 radius=0.15; visual cylinder length=0.1 radius=0.15
- added link rear_right_wheel; collision cylinder length=0.1 radius=0.15; visual cylinder length=0.1 radius=0.15
- link base_link: geometry collision box size=0.8 0.7 0.1; visual box size=0.8 0.7 0.1
Joints:
- added joint base_joint: type fixed, parent base_footprint, child base_link, origin xyz=0.0 0.0 0.135 rpy=0 0 0, axis 0.0 0.0 0.0
- added joint front_left_wheel_joint: type continuous, parent base_link, child front_left_wheel, origin xyz=-0.25 -0.4 0.0 rpy=1.57 0 0, axis 0.0 0.0 1.0
- added joint front_right_wheel_joint: type continuous, parent base_link, child front_right_wheel, origin xyz=-0.25 0.4 0.0 rpy=1.57 0 0, axis 0.0 0.0 1.0
- added joint rear_left_wheel_joint: type continuous, parent base_link, child rear_left_wheel, origin xyz=0.25 -0.4 0.0 rpy=1.57 0 0, axis 0.0 0.0 1.0
- added joint rear_right_wheel_joint: type continuous, parent base_link, child rear_right_wheel, origin xyz=0.25 0.4 0.0 rpy=1.57 0 0, axis 0.0 0.0 1.0
