Commit message: Cleanup and add .stl for tires

File: mobile_robot/urdf/rover.xacro (robot description, xacro)
@@ -36,9 +36,10 @@
         <axis xyz="0.0 0.0 0.0"/>
     </joint>
-    <xacro:macro name="wheel" params="name x y">
+    <xacro:macro name="wheel" params="name x y side">
         <link name="${name}_wheel_link">
             <visual>
                 <geometry>
                     <cylinder radius="0.15" length="0.1"/>
+                    <!-- <mesh filename="package://mobile_robot/meshes/left_tire.stl" scale="0.01 0.01 0.01"/> -->
                 </geometry>
                 <material name="black"/>
@@ -48,4 +49,5 @@
                 <geometry>
                     <cylinder radius="0.15" length="0.1"/>
+                    <!-- <mesh filename="package://mobile_robot/meshes/left_tire.stl" scale="0.01 0.01 0.01"/> -->
                 </geometry>
             </collision>
@@ -59,23 +61,23 @@
     </xacro:macro>
     <!-- Front Right Wheel -->
-    <xacro:wheel name="front_right" x="-0.25" y="0.4" />
+    <xacro:wheel name="front_right" x="-0.25" y="0.4" side="right"/>
     <!-- Rear Left Wheel -->
-    <xacro:wheel name="rear_left" x="0.25" y="-0.4" />
+    <xacro:wheel name="rear_left" x="0.25" y="-0.4" side="left"/>
     <!-- Rear Right Wheel -->
-    <xacro:wheel name="rear_right" x="0.25" y="0.4" />
+    <xacro:wheel name="rear_right" x="0.25" y="0.4" side="right"/>
     <xacro:property name="side" value="front_left"/>
     <!-- Front Left Wheel -->
     <link name="${side}_wheel_link">
         <visual>
-        <geometry>
-            <cylinder radius="0.15" length="0.1"/>
-        </geometry>
-        <material name="black"/>
+            <geometry>
+                <cylinder radius="0.15" length="0.1"/>
+            </geometry>
+            <material name="black"/>
         </visual>
         <collision>
-        <origin xyz="0.0 0.0 0.0" rpy="0.0 0.0 0.0"/>
-        <geometry>
-            <cylinder radius="0.15" length="0.1"/>
-        </geometry>
+            <origin xyz="0.0 0.0 0.0" rpy="0.0 0.0 0.0"/>
+            <geometry>
+                <cylinder radius="0.15" length="0.1"/>
+            </geometry>
         </collision>
     </link>

Commit message: Basic gazebo launch

File: mobile_robot/urdf/rover.xacro (robot description, xacro)
@@ -18,15 +18,22 @@
     <link name="base_link">
         <visual>
-        <geometry>
-            <box size="0.8 0.7 0.1"/>
-        </geometry>
-        <material name="blue"/>
+            <geometry>
+                <box size="0.8 0.7 0.1"/>
+            </geometry>
+            <material name="blue"/>
         </visual>
         <collision>
-        <origin xyz="0.0 0.0 0.0" rpy="0.0 0.0 0.0"/>
-        <geometry>
-            <box size="0.8 0.7 0.1"/>
-        </geometry>
+            <origin xyz="0.0 0.0 0.0" rpy="0.0 0.0 0.0"/>
+            <geometry>
+                <box size="0.8 0.7 0.1"/>
+            </geometry>
         </collision>
+        <inertial>
+                <origin xyz="0.0 0.0 0.0" rpy="0.0 0.0 0.0"/>
+                <mass value="1.0"/>
+                <inertia ixx="0.4" ixy="0.0" ixz="0.0"
+                        iyy="0.4" iyz="0.0"
+                        izz="0.2"/>
+            </inertial>
     </link>
     <joint name="base_joint" type="fixed">
@@ -52,4 +59,9 @@
                 </geometry>
             </collision>
+            <inertial>
+                <origin xyz="0.0 0.0 0.0" rpy="0.0 0.0 0.0"/>
+                <mass value="0.5"/>
+                <inertia ixx="0.0" ixy="0.0" ixz="0.0" iyy="0.0" iyz="0.0" izz="0.0"/>
+            </inertial>
         </link>
         <joint name="${name}_wheel_joint" type="continuous">
@@ -81,4 +93,9 @@
             </geometry>
         </collision>
+        <inertial>
+            <origin xyz="0.0 0.0 0.0" rpy="0.0 0.0 0.0"/>
+            <mass value="0.5"/>
+            <inertia ixx="0.0" ixy="0.0" ixz="0.0" iyy="0.0" iyz="0.0" izz="0.0"/>
+        </inertial>
     </link>
     <joint name="${side}_wheel_joint" type="continuous">

Commit message: Updated with intertia calcs

File: mobile_robot/urdf/rover.xacro (robot description, xacro)
@@ -14,5 +14,13 @@
     <color rgba="1 0 0 1"/>
   </material>
-  <link name="base_footprint"/>
+    <link name="base_footprint"/>
+    <xacro:property name="constant" value="${1.0/12.0}"/>
+    <xacro:property name="mass"     value="1.0"/>
+    <xacro:property name="width"    value="0.8"/>
+    <xacro:property name="width_sq"   value="${width*width}"/>
+    <xacro:property name="height"   value="0.1"/>
+    <xacro:property name="height_sq"   value="${height*height}"/>
+    <xacro:property name="depth"    value="0.7"/>
+    <xacro:property name="depth_sq"   value="${depth*depth}"/>
     <!-- Body-->
     <link name="base_link">
@@ -26,5 +34,5 @@
             <origin xyz="0.0 0.0 0.0" rpy="0.0 0.0 0.0"/>
             <geometry>
-                <box size="0.8 0.7 0.1"/>
+                <box size="${width} ${depth} ${height}"/>
             </geometry>
         </collision>
@@ -32,7 +40,7 @@
                 <origin xyz="0.0 0.0 0.0" rpy="0.0 0.0 0.0"/>
                 <mass value="1.0"/>
-                <inertia ixx="0.4" ixy="0.0" ixz="0.0"
-                        iyy="0.4" iyz="0.0"
-                        izz="0.2"/>
+                <inertia ixx="${constant*mass*(height_sq + depth_sq) }" ixy="0.0" ixz="0.0"
+                                   iyy="${constant*mass*(width*width + height*height)}" iyz="0.0"
+                                             izz="${constant*mass*(width*width + depth*depth)}"/>
             </inertial>
     </link>
@@ -45,18 +53,4 @@
     <xacro:macro name="wheel" params="name x y side">
         <link name="${name}_wheel_link">
-            <visual>
-                <geometry>
-                    <cylinder radius="0.15" length="0.1"/>
-                    <!-- <mesh filename="package://mobile_robot/meshes/left_tire.stl" scale="0.01 0.01 0.01"/> -->
-                </geometry>
-                <material name="black"/>
-            </visual>
-            <collision>
-                <origin xyz="0.0 0.0 0.0" rpy="0.0 0.0 0.0"/>
-                <geometry>
-                    <cylinder radius="0.15" length="0.1"/>
-                    <!-- <mesh filename="package://mobile_robot/meshes/left_tire.stl" scale="0.01 0.01 0.01"/> -->
-                </geometry>
-            </collision>
             <inertial>
                 <origin xyz="0.0 0.0 0.0" rpy="0.0 0.0 0.0"/>
@@ -64,9 +58,25 @@
                 <inertia ixx="0.0" ixy="0.0" ixz="0.0" iyy="0.0" iyz="0.0" izz="0.0"/>
             </inertial>
+            <visual name="">
+                <origin xyz="0.0 0.0 0.0" rpy="0.0 0.0 0.0"/>
+                <geometry>
+                    <mesh filename="package://mobile_robot/meshes/${side}_tire.dae" scale="0.005 0.005 0.005"/>
+                </geometry>
+                <material name="black">
+                    <color rgba=".0 .0 0.0 1.0"/>
+                </material>
+            </visual>
+            <collision>
+                <origin xyz="0.0 0.0 0.0" rpy="0.0 0.0 0.0"/>
+                <geometry>
+                    <mesh filename="package://mobile_robot/meshes/${side}_tire.dae" scale="0.005 0.005 0.005"/>
+                </geometry>
+            </collision>
         </link>
         <joint name="${name}_wheel_joint" type="continuous">
             <parent link="base_link"/>
             <child link="${name}_wheel_link"/>
-            <origin rpy="1.57 0 0" xyz="${x} ${y} 0.0"/>
+            <!-- <origin rpy="1.57 0 0" xyz="${x} ${y} 0.0"/> -->
+            <origin rpy="0 0 0" xyz="${x} ${y} 0.0"/>
             <axis xyz="0.0 0.0 1.0"/>
         </joint>
@@ -83,5 +93,6 @@
         <visual>
             <geometry>
-                <cylinder radius="0.15" length="0.1"/>
+                <!-- <cylinder radius="0.15" length="0.1"/> -->
+                <mesh filename="package://mobile_robot/meshes/left_tire.stl" scale="0.005 0.005 0.005"/>
             </geometry>
             <material name="black"/>
@@ -90,5 +101,6 @@
             <origin xyz="0.0 0.0 0.0" rpy="0.0 0.0 0.0"/>
             <geometry>
-                <cylinder radius="0.15" length="0.1"/>
+                <!-- <cylinder radius="0.15" length="0.1"/> -->
+                <mesh filename="package://mobile_robot/meshes/left_tire.stl" scale="0.005 0.005 0.005"/>
             </geometry>
         </collision>
@@ -96,5 +108,7 @@
             <origin xyz="0.0 0.0 0.0" rpy="0.0 0.0 0.0"/>
             <mass value="0.5"/>
-            <inertia ixx="0.0" ixy="0.0" ixz="0.0" iyy="0.0" iyz="0.0" izz="0.0"/>
+            <inertia ixx="0.0" ixy="0.0" ixz="0.0"
+                    iyy="0.0" iyz="0.0"
+                                    izz="0.0"/>
         </inertial>
     </link>
@@ -102,5 +116,6 @@
         <parent link="base_link"/>
         <child link="${side}_wheel_link"/>
-        <origin rpy="1.57 0 0" xyz="-0.25 -0.4 0.0"/>
+        <!-- <origin rpy="1.57 0 0" xyz="-0.25 -0.4 0.0"/> -->
+        <origin rpy="0 0 0" xyz="-0.25 -0.4 0.0"/>
         <axis xyz="0.0 0.0 1.0"/>
     </joint>

Commit message: Lab10 update to match exactly to video

File: mobile_robot/urdf/rover.xacro (robot description, xacro)
@@ -29,5 +29,5 @@
                 <box size="0.8 0.7 0.1"/>
             </geometry>
-            <material name="blue"/>
+            <material name="red"/>
         </visual>
         <collision>
@@ -52,5 +52,5 @@
     </joint>
     <xacro:macro name="wheel" params="name x y side">
-        <link name="${name}_wheel_link">
+        <link name="${name}_link">
             <inertial>
                 <origin xyz="0.0 0.0 0.0" rpy="0.0 0.0 0.0"/>
@@ -61,62 +61,30 @@
                 <origin xyz="0.0 0.0 0.0" rpy="0.0 0.0 0.0"/>
                 <geometry>
-                    <mesh filename="package://mobile_robot/meshes/${side}_tire.dae" scale="0.005 0.005 0.005"/>
+                    <mesh filename="package://mobile_robot/meshes/${side}_tire.stl" scale="0.005 0.005 0.005"/>
                 </geometry>
-                <material name="black">
-                    <color rgba=".0 .0 0.0 1.0"/>
-                </material>
+                <material name="black"/>
             </visual>
             <collision>
                 <origin xyz="0.0 0.0 0.0" rpy="0.0 0.0 0.0"/>
                 <geometry>
-                    <mesh filename="package://mobile_robot/meshes/${side}_tire.dae" scale="0.005 0.005 0.005"/>
+                    <mesh filename="package://mobile_robot/meshes/${side}_tire.stl" scale="0.005 0.005 0.005"/>
                 </geometry>
             </collision>
         </link>
-        <joint name="${name}_wheel_joint" type="continuous">
+        <joint name="${name}_joint" type="continuous">
             <parent link="base_link"/>
-            <child link="${name}_wheel_link"/>
+            <child link="${name}_link"/>
             <!-- <origin rpy="1.57 0 0" xyz="${x} ${y} 0.0"/> -->
             <origin rpy="0 0 0" xyz="${x} ${y} 0.0"/>
-            <axis xyz="0.0 0.0 1.0"/>
+            <axis xyz="0.0 1.0 0.0"/>
         </joint>
     </xacro:macro>
     <!-- Front Right Wheel -->
-    <xacro:wheel name="front_right" x="-0.25" y="0.4" side="right"/>
+    <xacro:wheel name="wheel_front_right" x="-0.25" y="0.4" side="right"/>
     <!-- Rear Left Wheel -->
-    <xacro:wheel name="rear_left" x="0.25" y="-0.4" side="left"/>
+    <xacro:wheel name="wheel_rear_left" x="0.25" y="-0.4" side="left"/>
     <!-- Rear Right Wheel -->
-    <xacro:wheel name="rear_right" x="0.25" y="0.4" side="right"/>
-    <xacro:property name="side" value="front_left"/>
+    <xacro:wheel name="wheel_rear_right" x="0.25" y="0.4" side="right"/>
     <!-- Front Left Wheel -->
-    <link name="${side}_wheel_link">
-        <visual>
-            <geometry>
-                <!-- <cylinder radius="0.15" length="0.1"/> -->
-                <mesh filename="package://mobile_robot/meshes/left_tire.stl" scale="0.005 0.005 0.005"/>
-            </geometry>
-            <material name="black"/>
-        </visual>
-        <collision>
-            <origin xyz="0.0 0.0 0.0" rpy="0.0 0.0 0.0"/>
-            <geometry>
-                <!-- <cylinder radius="0.15" length="0.1"/> -->
-                <mesh filename="package://mobile_robot/meshes/left_tire.stl" scale="0.005 0.005 0.005"/>
-            </geometry>
-        </collision>
-        <inertial>
-            <origin xyz="0.0 0.0 0.0" rpy="0.0 0.0 0.0"/>
-            <mass value="0.5"/>
-            <inertia ixx="0.0" ixy="0.0" ixz="0.0"
-                    iyy="0.0" iyz="0.0"
-                                    izz="0.0"/>
-        </inertial>
-    </link>
-    <joint name="${side}_wheel_joint" type="continuous">
-        <parent link="base_link"/>
-        <child link="${side}_wheel_link"/>
-        <!-- <origin rpy="1.57 0 0" xyz="-0.25 -0.4 0.0"/> -->
-        <origin rpy="0 0 0" xyz="-0.25 -0.4 0.0"/>
-        <axis xyz="0.0 0.0 1.0"/>
-    </joint>
+    <xacro:wheel name="wheel_front_left" x="-0.25" y="-0.4" side="left"/>
 </robot>
