Commit message: Simple display of rear pole

File: urdf_sim_tutorial/urdf/14-gripper.urdf.xacro (robot description, xacro)
@@ -139,4 +139,27 @@
     </joint>
   </transmission>
+  <link name="gripper_pole_back">
+      <visual>
+        <geometry>
+          <cylinder length="${-1*polelen}" radius="0.01"/>
+        </geometry>
+        <origin xyz="${-1*polelen/2} 0 0" rpy="0 ${pi/2} 0 "/>
+      </visual>
+      <collision>
+        <geometry>
+          <cylinder length="${-1*polelen}" radius="0.01"/>
+        </geometry>
+        <origin xyz="${-1*polelen/2} 0 0" rpy="0 ${pi/2} 0 "/>
+      </collision>
+      <xacro:default_inertial mass="0.05"/>
+  </link>
+  <joint name="gripper_extension_back" type="prismatic">
+    <parent link="base_link"/>
+    <child link="gripper_pole_back"/>
+    <limit effort="1000.0" lower="-${width*2-.02}" upper="0" velocity="0.5"/>
+    <origin rpy="0 0 0" xyz="${-1*width-.01} 0 0.2"/>
+    <limit effort="30" velocity="0.2"/>
+    <dynamics damping="0.0" friction="0.0"/>
+  </joint>
   <xacro:macro name="gripper" params="prefix reflect">
     <joint name="${prefix}_gripper_joint" type="revolute">

Commit message: Enable back pole

File: urdf_sim_tutorial/urdf/14-gripper.urdf.xacro (robot description, xacro)
@@ -142,5 +142,5 @@
       <visual>
         <geometry>
-          <cylinder length="${-1*polelen}" radius="0.01"/>
+          <cylinder length="${polelen}" radius="0.01"/>
         </geometry>
         <origin xyz="${-1*polelen/2} 0 0" rpy="0 ${pi/2} 0 "/>
@@ -148,5 +148,5 @@
       <collision>
         <geometry>
-          <cylinder length="${-1*polelen}" radius="0.01"/>
+          <cylinder length="${polelen}" radius="0.01"/>
         </geometry>
         <origin xyz="${-1*polelen/2} 0 0" rpy="0 ${pi/2} 0 "/>
@@ -157,20 +157,20 @@
     <parent link="base_link"/>
     <child link="gripper_pole_back"/>
-    <limit effort="1000.0" lower="-${width*2-.02}" upper="0" velocity="0.5"/>
-    <origin rpy="0 0 0" xyz="${-1*width-.01} 0 0.2"/>
+    <limit effort="1000.0" lower="${width*2-.02}" upper="0" velocity="0.5"/>
+    <origin rpy="0 0 0" xyz="${-1*width+.01} 0 0.2"/>
     <limit effort="30" velocity="0.2"/>
     <dynamics damping="0.0" friction="0.0"/>
   </joint>
-  <xacro:macro name="gripper" params="prefix reflect">
-    <joint name="${prefix}_gripper_joint" type="revolute">
+ <xacro:macro name="gripper" params="prefix suffix reflect front1_back0">
+    <joint name="${prefix}_gripper_joint_${suffix}" type="revolute">
       <axis xyz="0 0 ${reflect}"/>
       <limit effort="1000.0" lower="0.0" upper="0.548" velocity="0.5"/>
-      <origin rpy="0 0 0" xyz="${polelen} ${reflect*0.01} 0"/>
+      <origin rpy="0 0 0" xyz="${front1_back0*polelen} ${reflect*0.01} 0"/>
       <parent link="gripper_pole"/>
-      <child link="${prefix}_gripper"/>
+      <child link="${prefix}_gripper_${suffix}"/>
       <limit effort="30" velocity="1.0"/>
       <dynamics damping="0.0" friction="0.0"/>
     </joint>
-    <link name="${prefix}_gripper">
+    <link name="${prefix}_gripper_${suffix}">
       <visual>
         <origin rpy="${(reflect-1)/2*pi} 0 0" xyz="0 0 0"/>
@@ -187,18 +187,18 @@
       <xacro:default_inertial mass="0.05"/>
     </link>
-    <transmission name="${prefix}_gripper_trans" type="SimpleTransmission">
+    <transmission name="${prefix}_gripper_trans_${suffix}" type="SimpleTransmission">
       <type>transmission_interface/SimpleTransmission</type>
-      <actuator name="${prefix}_gripper_motor">
+      <actuator name="${prefix}_gripper_motor_${suffix}">
         <mechanicalReduction>1</mechanicalReduction>
       </actuator>
-      <joint name="${prefix}_gripper_joint">
+      <joint name="${prefix}_gripper_joint_${suffix}">
         <hardwareInterface>PositionJointInterface</hardwareInterface>
       </joint>
     </transmission>
-    <joint name="${prefix}_tip_joint" type="fixed">
-      <parent link="${prefix}_gripper"/>
-      <child link="${prefix}_tip"/>
-    </joint>
-    <link name="${prefix}_tip">
+    <joint name="${prefix}_tip_joint_${suffix}" type="fixed">
+      <parent link="${prefix}_gripper_${suffix}"/>
+      <child link="${prefix}_tip_${suffix}"/>
+    </joint>
+    <link name="${prefix}_tip_${suffix}">
       <visual>
         <origin rpy="${(reflect-1)/2*pi} 0 0" xyz="0.09137 0.00495 0"/>
@@ -216,6 +216,6 @@
     </link>
   </xacro:macro>
-  <xacro:gripper prefix="left" reflect="1" />
-  <xacro:gripper prefix="right" reflect="-1" />
+  <xacro:gripper prefix="left" suffix="front" reflect="1" front1_back0="1"/>
+  <!-- <xacro:gripper prefix="right" suffix="front" reflect="-1" front1_back0="1"/> -->
   <link name="head">
     <visual>

Commit message: Complerted back gripper

File: urdf_sim_tutorial/urdf/14-gripper.urdf.xacro (robot description, xacro)
@@ -109,5 +109,5 @@
   <joint name="gripper_extension" type="prismatic">
     <parent link="base_link"/>
-    <child link="gripper_pole"/>
+    <child link="gripper_pole_front"/>
     <limit effort="1000.0" lower="-${width*2-.02}" upper="0" velocity="0.5"/>
     <origin rpy="0 0 0" xyz="${width-.01} 0 0.2"/>
@@ -115,5 +115,5 @@
     <dynamics damping="0.0" friction="0.0"/>
   </joint>
-  <link name="gripper_pole">
+  <link name="gripper_pole_front">
     <visual>
       <geometry>
@@ -157,15 +157,15 @@
     <parent link="base_link"/>
     <child link="gripper_pole_back"/>
-    <limit effort="1000.0" lower="${width*2-.02}" upper="0" velocity="0.5"/>
+    <limit effort="1000.0" upper="${width*2-.02}" lower="0" velocity="0.5"/>
     <origin rpy="0 0 0" xyz="${-1*width+.01} 0 0.2"/>
     <limit effort="30" velocity="0.2"/>
     <dynamics damping="0.0" friction="0.0"/>
   </joint>
- <xacro:macro name="gripper" params="prefix suffix reflect front1_back0">
+ <xacro:macro name="gripper" params="prefix suffix reflect front1_back0 reflectY">
     <joint name="${prefix}_gripper_joint_${suffix}" type="revolute">
       <axis xyz="0 0 ${reflect}"/>
-      <limit effort="1000.0" lower="0.0" upper="0.548" velocity="0.5"/>
+      <limit effort="1000.0" lower="0.0" upper="${0.548*reflectY}" velocity="0.5"/>
       <origin rpy="0 0 0" xyz="${front1_back0*polelen} ${reflect*0.01} 0"/>
-      <parent link="gripper_pole"/>
+      <parent link="gripper_pole_${suffix}"/>
       <child link="${prefix}_gripper_${suffix}"/>
       <limit effort="30" velocity="1.0"/>
@@ -174,5 +174,5 @@
     <link name="${prefix}_gripper_${suffix}">
       <visual>
-        <origin rpy="${(reflect-1)/2*pi} 0 0" xyz="0 0 0"/>
+        <origin rpy="${(reflect-1)/2*pi} ${(reflectY-1)/2*pi} 0" xyz="0 0 0"/>
         <geometry>
           <mesh filename="package://urdf_tutorial/meshes/l_finger.dae"/>
@@ -183,5 +183,5 @@
           <mesh filename="package://urdf_tutorial/meshes/l_finger.dae"/>
         </geometry>
-        <origin rpy="${(reflect-1)/2*pi} 0 0" xyz="0 0 0"/>
+        <origin rpy="${(reflect-1)/2*pi} ${(reflectY-1)/2*pi} 0" xyz="0 0 0"/>
       </collision>
       <xacro:default_inertial mass="0.05"/>
@@ -202,5 +202,5 @@
     <link name="${prefix}_tip_${suffix}">
       <visual>
-        <origin rpy="${(reflect-1)/2*pi} 0 0" xyz="0.09137 0.00495 0"/>
+        <origin rpy="${(reflect-1)/2*pi} ${(reflectY-1)/2*pi} 0" xyz="${0.09137*reflectY} ${0.00495*reflectY} 0"/>
         <geometry>
           <mesh filename="package://urdf_tutorial/meshes/l_finger_tip.dae"/>
@@ -211,11 +211,13 @@
           <mesh filename="package://urdf_tutorial/meshes/l_finger_tip.dae"/>
         </geometry>
-        <origin rpy="${(reflect-1)/2*pi} 0 0" xyz="0.09137 0.00495 0"/>
+        <origin rpy="${(reflect-1)/2*pi} ${(reflectY-1)/2*pi} 0" xyz="${0.09137*reflectY} ${0.00495*reflectY} 0"/>
       </collision>
       <xacro:default_inertial mass="0.05"/>
     </link>
   </xacro:macro>
-  <xacro:gripper prefix="left" suffix="front" reflect="1" front1_back0="1"/>
-  <!-- <xacro:gripper prefix="right" suffix="front" reflect="-1" front1_back0="1"/> -->
+  <xacro:gripper prefix="left" suffix="front" reflect="1" front1_back0="1" reflectY="1"/>
+  <xacro:gripper prefix="right" suffix="front" reflect="-1" front1_back0="1" reflectY="1"/>
+  <xacro:gripper prefix="left" suffix="back" reflect="1" front1_back0="-1" reflectY="-1"/>
+  <xacro:gripper prefix="right" suffix="back" reflect="-1" front1_back0="-1" reflectY="-1"/>
   <link name="head">
     <visual>

Commit message: Completed lab11

File: urdf_sim_tutorial/urdf/14-gripper.urdf.xacro (robot description, xacro)
@@ -107,5 +107,5 @@
   <xacro:leg prefix="right" reflect="-1" />
   <xacro:leg prefix="left" reflect="1" />
-  <joint name="gripper_extension" type="prismatic">
+  <joint name="gripper_extension_front" type="prismatic">
     <parent link="base_link"/>
     <child link="gripper_pole_front"/>
@@ -135,5 +135,5 @@
       <mechanicalReduction>1</mechanicalReduction>
     </actuator>
-    <joint name="gripper_extension">
+    <joint name="gripper_extension_front">
       <hardwareInterface>PositionJointInterface</hardwareInterface>
     </joint>
@@ -162,9 +162,18 @@
     <dynamics damping="0.0" friction="0.0"/>
   </joint>
- <xacro:macro name="gripper" params="prefix suffix reflect front1_back0 reflectY">
+  <transmission name="gripper_extension_trans_back" type="SimpleTransmission">
+    <type>transmission_interface/SimpleTransmission</type>
+    <actuator name="gripper_extension_motor_back">
+      <mechanicalReduction>1</mechanicalReduction>
+    </actuator>
+    <joint name="gripper_extension_back">
+      <hardwareInterface>PositionJointInterface</hardwareInterface>
+    </joint>
+  </transmission>
+ <xacro:macro name="gripper" params="prefix suffix reflect reflectY">
     <joint name="${prefix}_gripper_joint_${suffix}" type="revolute">
       <axis xyz="0 0 ${reflect}"/>
       <limit effort="1000.0" lower="0.0" upper="${0.548*reflectY}" velocity="0.5"/>
-      <origin rpy="0 0 0" xyz="${front1_back0*polelen} ${reflect*0.01} 0"/>
+      <origin rpy="0 0 0" xyz="${reflectY*polelen} ${reflect*0.01} 0"/>
       <parent link="gripper_pole_${suffix}"/>
       <child link="${prefix}_gripper_${suffix}"/>
@@ -216,8 +225,8 @@
     </link>
   </xacro:macro>
-  <xacro:gripper prefix="left" suffix="front" reflect="1" front1_back0="1" reflectY="1"/>
-  <xacro:gripper prefix="right" suffix="front" reflect="-1" front1_back0="1" reflectY="1"/>
-  <xacro:gripper prefix="left" suffix="back" reflect="1" front1_back0="-1" reflectY="-1"/>
-  <xacro:gripper prefix="right" suffix="back" reflect="-1" front1_back0="-1" reflectY="-1"/>
+  <xacro:gripper prefix="left" suffix="front" reflect="1" reflectY="1"/>
+  <xacro:gripper prefix="right" suffix="front" reflect="-1" reflectY="1"/>
+  <xacro:gripper prefix="left" suffix="back" reflect="1" reflectY="-1"/>
+  <xacro:gripper prefix="right" suffix="back" reflect="-1"  reflectY="-1"/>
   <link name="head">
     <visual>
