Commit message: Lab11 add notes and commands; enhance to drive

File: urdf_sim_tutorial/urdf/12-gripper.urdf.xacro (robot description, xacro)
@@ -107,5 +107,5 @@
   <xacro:leg prefix="right" reflect="-1" />
   <xacro:leg prefix="left" reflect="1" />
-  <joint name="gripper_extension" type="prismatic">
+  <joint name="gripper_extension_front" type="prismatic">
     <parent link="base_link"/>
     <child link="gripper_pole"/>
@@ -135,5 +135,5 @@
       <mechanicalReduction>1</mechanicalReduction>
     </actuator>
-    <joint name="gripper_extension">
+    <joint name="gripper_extension_front">
       <hardwareInterface>PositionJointInterface</hardwareInterface>
     </joint>

File: urdf_sim_tutorial/urdf/14-gripper.urdf.xacro (robot description, xacro)
@@ -60,4 +60,24 @@
       <origin xyz="${baselen*reflect/3} 0 -${wheeldiam/2+.05}" rpy="0 0 0"/>
     </joint>
+    <!-- This block provides the simulator (Gazebo) with information on a few additional
+    physical properties. See http://gazebosim.org/tutorials/?tut=ros_urdf for more-->
+    <gazebo reference="${prefix}_${suffix}_wheel">
+      <mu1 value="200.0"/>
+      <mu2 value="100.0"/>
+      <kp value="10000000.0" />
+      <kd value="1.0" />
+      <material>Gazebo/Grey</material>
+    </gazebo>
+    <!-- This block connects the wheel joint to an actuator (motor), which informs both
+    simulation and visualization of the robot -->
+    <transmission name="${prefix}_${suffix}_wheel_trans">
+      <type>transmission_interface/SimpleTransmission</type>
+      <actuator name="${prefix}_${suffix}_wheel_motor">
+        <mechanicalReduction>1</mechanicalReduction>
+      </actuator>
+      <joint name="${prefix}_${suffix}_wheel_joint">
+        <hardwareInterface>VelocityJointInterface</hardwareInterface>
+      </joint>
+    </transmission>
   </xacro:macro>
   <xacro:macro name="leg" params="prefix reflect">
