Commit message: Lab14 completed

File: universal_robot/ur_description/urdf/ur5.urdf.xacro (robot description, xacro)
@@ -12,4 +12,14 @@
     </inertial>
   </xacro:macro>
+  <!-- <xacro:macro name="ur5_robot" params="prefix joint_limited
+    shoulder_pan_lower_limit:=${-pi}    shoulder_pan_upper_limit:=${pi}
+    shoulder_lift_lower_limit:=${-pi}    shoulder_lift_upper_limit:=${pi}
+    elbow_joint_lower_limit:=${-pi}    elbow_joint_upper_limit:=${pi}
+    wrist_1_lower_limit:=${-pi}    wrist_1_upper_limit:=${pi}
+    wrist_2_lower_limit:=${-pi}    wrist_2_upper_limit:=${pi}
+    wrist_3_lower_limit:=${-pi}    wrist_3_upper_limit:=${pi}
+    transmission_hw_interface:=hardware_interface/EffortJointInterface
+    safety_limits:=false safety_pos_margin:=0.15
+    safety_k_position:=20"> -->
   <xacro:macro name="ur5_robot" params="prefix joint_limited
     shoulder_pan_lower_limit:=${-pi}    shoulder_pan_upper_limit:=${pi}
